File: attiny861a_breakout/attiny861a_breakout.sch (KiCad schematic (older format))
At the start: 8 parts, among them IC1 ATTINY861A-S

Commit message: switched reset pullups from 2K2 to 10K
Parts:
- R1: value 2K2 -> 10K
Changed lines of the file:
@@
 $EndComp
 $Comp
-L +5V #PWR1
+L +5V #PWR01
 U 1 1 58E29592
 P 3400 2800
-F 0 "#PWR1" H 3400 2650 50  0001 C CNN
+F 0 "#PWR01" H 3400 2650 50  0001 C CNN
 F 1 "+5V" H 3400 2940 50  0000 C CNN
 F 2 "" H 3400 2800 50  0000 C CNN
@@
 $EndComp
 $Comp
-L GND #PWR2
+L GND #PWR02
 U 1 1 58E295D6
 P 3400 4700
-F 0 "#PWR2" H 3400 4450 50  0001 C CNN
+F 0 "#PWR02" H 3400 4450 50  0001 C CNN
 F 1 "GND" H 3400 4550 50  0000 C CNN
 F 2 "" H 3400 4700 50  0000 C CNN
@@
 SDA
 $Comp
-L GND #PWR6
+L GND #PWR03
 U 1 1 58E323E4
 P 6450 5350
-F 0 "#PWR6" H 6450 5100 50  0001 C CNN
+F 0 "#PWR03" H 6450 5100 50  0001 C CNN
 F 1 "GND" H 6450 5200 50  0000 C CNN
 F 2 "" H 6450 5350 50  0000 C CNN
@@
 $EndComp
 $Comp
-L +5V #PWR7
+L +5V #PWR04
 U 1 1 58E326D5
 P 6550 5150
-F 0 "#PWR7" H 6550 5000 50  0001 C CNN
+F 0 "#PWR04" H 6550 5000 50  0001 C CNN
 F 1 "+5V" H 6550 5290 50  0000 C CNN
 F 2 "" H 6550 5150 50  0000 C CNN
@@
 $EndComp
 $Comp
-L GND #PWR9
+L GND #PWR05
 U 1 1 58E39CFA
 P 7750 5000
-F 0 "#PWR9" H 7750 4750 50  0001 C CNN
+F 0 "#PWR05" H 7750 4750 50  0001 C CNN
 F 1 "GND" H 7750 4850 50  0000 C CNN
 F 2 "" H 7750 5000 50  0000 C CNN
@@
 $EndComp
 $Comp
-L +5V #PWR8
+L +5V #PWR06
 U 1 1 58E39D32
 P 7550 5000
-F 0 "#PWR8" H 7550 4850 50  0001 C CNN
+F 0 "#PWR06" H 7550 4850 50  0001 C CNN
 F 1 "+5V" H 7550 5140 50  0000 C CNN
 F 2 "" H 7550 5000 50  0000 C CNN
@@
 	5850 2900 5600 2900
 Wire Wire Line
-	5600 3800 6800 3800
+	5600 3800 6150 3800
+Wire Wire Line
+	6150 3800 6800 3800
 Wire Wire Line
 	6150 3800 6150 4900
@@
 	5800 5150 5950 5150
 Wire Wire Line
-	5600 4000 6750 4000
+	5600 4000 6050 4000
+Wire Wire Line
+	6050 4000 6750 4000
 Wire Wire Line
 	6050 4000 6050 4850
@@
 	5700 4500 5700 5350
 Wire Wire Line
-	5350 5350 5950 5350
-Wire Wire Line
-	5600 3200 7750 3200
+	5350 5350 5700 5350
+Wire Wire Line
+	5700 5350 5950 5350
+Wire Wire Line
+	5600 3200 7400 3200
+Wire Wire Line
+	7400 3200 7750 3200
 Connection ~ 6050 4000
 Wire Wire Line
@@
 	6050 3000 6050 3150
 Wire Wire Line
-	6050 3150 7750 3150
+	6050 3150 7450 3150
+Wire Wire Line
+	7450 3150 7750 3150
 Wire Wire Line
 	7750 3150 7750 3100
@@
 	5900 3300 5900 3250
 Wire Wire Line
-	5900 3250 7750 3250
+	5900 3250 7350 3250
+Wire Wire Line
+	7350 3250 7750 3250
 Wire Wire Line
 	7750 3250 7750 3300
@@
 	5950 3400 5950 3300
 Wire Wire Line
-	5950 3300 7700 3300
+	5950 3300 7300 3300
+Wire Wire Line
+	7300 3300 7700 3300
 Wire Wire Line
 	7700 3300 7700 3400
@@
 	6000 3500 6000 3350
 Wire Wire Line
-	6000 3350 7650 3350
+	6000 3350 7250 3350
+Wire Wire Line
+	7250 3350 7650 3350
 Wire Wire Line
 	7650 3350 7650 3500
@@
 	6050 3600 6050 3400
 Wire Wire Line
-	6050 3400 7600 3400
+	6050 3400 7200 3400
+Wire Wire Line
+	7200 3400 7600 3400
 Wire Wire Line
 	7600 3400 7600 3600
@@
 	7600 3600 7750 3600
 Wire Wire Line
-	5600 3900 6500 3900
+	5600 3900 6100 3900
+Wire Wire Line
+	6100 3900 6500 3900
 Wire Wire Line
 	5600 4400 6850 4400
@@
 	6500 2400 7700 2400
 $Comp
-L +5V #PWR4
+L +5V #PWR07
 U 1 1 58E561FB
 P 6200 1200
-F 0 "#PWR4" H 6200 1050 50  0001 C CNN
+F 0 "#PWR07" H 6200 1050 50  0001 C CNN
 F 1 "+5V" H 6200 1340 50  0000 C CNN
 F 2 "" H 6200 1200 50  0000 C CNN
@@
 $EndComp
 $Comp
-L GND #PWR5
+L GND #PWR08
 U 1 1 58E5624E
 P 6200 1700
-F 0 "#PWR5" H 6200 1450 50  0001 C CNN
+F 0 "#PWR08" H 6200 1450 50  0001 C CNN
 F 1 "GND" H 6200 1550 50  0000 C CNN
 F 2 "" H 6200 1700 50  0000 C CNN
@@
 	5900 1300 5900 3100
 Wire Wire Line
-	3400 2800 3400 3300
+	3400 2800 3400 2900
+Wire Wire Line
+	3400 2900 3400 3300
 Connection ~ 3400 2900
 Wire Wire Line
-	3400 4100 3400 4700
+	3400 4100 3400 4500
+Wire Wire Line
+	3400 4500 3400 4700
 Connection ~ 3400 4500
 Wire Wire Line
@@
 P 5350 5200
 F 0 "R1" V 5430 5200 50  0000 C CNN
-F 1 "2K2" V 5350 5200 50  0000 C CNN
+F 1 "10K" V 5350 5200 50  0000 C CNN
 F 2 "Resistors_SMD:R_0805" V 5500 5200 50  0000 C CNN
 F 3 "" H 5350 5200 50  0000 C CNN
@@
 Connection ~ 5700 5350
 $Comp
-L +5V #PWR3
+L +5V #PWR09
 U 1 1 58E6B644
 P 5350 4950
-F 0 "#PWR3" H 5350 4800 50  0001 C CNN
+F 0 "#PWR09" H 5350 4800 50  0001 C CNN
 F 1 "+5V" H 5350 5090 50  0000 C CNN
 F 2 "" H 5350 4950 50  0000 C CNN
