File: attiny861a_breakout/attiny861a_breakout.kicad_pcb (KiCad board)
At the start: 2 copper layers, 16 x 29 mm, 8 parts, among them IC1 ATTINY861A-S

Commit message: bugfixing
Routing:
- net /SCL_2: track 22.3 -> 20.2 mm
Changed lines of the file:
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@@
   (general
     (links 37)
-    (no_connects 0)
-    (area 41.924999 44.924999 58.075001 74.075001)
+    (no_connects 1)
+    (area 40.974999 38.3 72.135715 89.000001)
     (thickness 1.6)
     (drawings 27)
@@
   )
   (setup
-    (last_trace_width 0.6)
+    (last_trace_width 0.25)
     (user_trace_width 0.6)
     (trace_clearance 0.2)
@@
   (gr_line (start 42 74) (end 58 74) (layer Edge.Cuts) (width 0.15))
   (gr_line (start 42 74) (end 42 69) (layer Edge.Cuts) (width 0.15))
+  (segment (start 43.015 72.54) (end 43.855 71.7) (width 0.25) (layer F.Cu) (net 1))
+  (segment (start 43.855 71.7) (end 44.9 71.7) (width 0.25) (layer F.Cu) (net 1))
+  (segment (start 44.9 71.7) (end 45.6 71) (width 0.25) (layer F.Cu) (net 1))
+  (segment (start 45.6 71) (end 45.6 69.574998) (width 0.25) (layer F.Cu) (net 1))
+  (segment (start 47.892998 67.282) (end 48.25 67.282) (width 0.25) (layer F.Cu) (net 1))
+  (segment (start 45.6 69.574998) (end 47.892998 67.282) (width 0.25) (layer F.Cu) (net 1))
   (segment (start 48.25 67.282) (end 50 67.282) (width 0.25) (layer F.Cu) (net 1))
-  (segment (start 45.737999 69.436999) (end 47.892998 67.282) (width 0.25) (layer F.Cu) (net 1))
-  (segment (start 47.892998 67.282) (end 48.25 67.282) (width 0.25) (layer F.Cu) (net 1))
-  (segment (start 43.776999 71.778001) (end 44.121999 71.778001) (width 0.25) (layer F.Cu) (net 1))
-  (segment (start 43.015 72.54) (end 43.776999 71.778001) (width 0.25) (layer F.Cu) (net 1))
-  (segment (start 44.121999 71.778001) (end 45.737999 70.162001) (width 0.25) (layer F.Cu) (net 1))
-  (segment (start 45.737999 70.162001) (end 45.737999 69.436999) (width 0.25) (layer F.Cu) (net 1))
   (segment (start 55.721561 62.696326) (end 56.02156 62.396327) (width 0.25) (layer F.Cu) (net 1))
   (segment (start 50 67.282) (end 51.517741 67.282) (width 0.25) (layer F.Cu) (net 1))
@@
   (via (at 56.02156 62.396327) (size 0.6) (drill 0.4) (layers F.Cu B.Cu) (net 1))
   (segment (start 54.7 62.66) (end 55.925 62.66) (width 0.25) (layer B.Cu) (net 1))
-  (segment (start 48.273 66.012) (end 50 66.012) (width 0.25) (layer F.Cu) (net 2))
-  (segment (start 44.285 70) (end 48.273 66.012) (width 0.25) (layer F.Cu) (net 2))
+  (segment (start 44.285 70) (end 44.4 70) (width 0.25) (layer F.Cu) (net 2))
+  (segment (start 44.4 70) (end 48.388 66.012) (width 0.25) (layer F.Cu) (net 2))
+  (segment (start 48.388 66.012) (end 50 66.012) (width 0.25) (layer F.Cu) (net 2))
   (segment (start 55.774991 59.899999) (end 56.07499 59.6) (width 0.25) (layer F.Cu) (net 2))
   (segment (start 51.75 66.012) (end 52.725021 65.036979) (width 0.25) (layer F.Cu) (net 2))
@@
   (via (at 56.000004 55) (size 0.6) (drill 0.4) (layers F.Cu B.Cu) (net 4))
   (segment (start 54.7 55.04) (end 55.960004 55.04) (width 0.25) (layer B.Cu) (net 4))
+  (segment (start 48.095 72.54) (end 48.856999 71.778001) (width 0.25) (layer B.Cu) (net 5))
+  (segment (start 51.700005 68.004211) (end 52.000004 67.704212) (width 0.25) (layer B.Cu) (net 5))
+  (segment (start 48.856999 71.778001) (end 49.721999 71.778001) (width 0.25) (layer B.Cu) (net 5))
+  (segment (start 49.721999 71.778001) (end 50.6 70.9) (width 0.25) (layer B.Cu) (net 5))
+  (segment (start 50.6 70.9) (end 50.6 69.104216) (width 0.25) (layer B.Cu) (net 5))
+  (segment (start 50.6 69.104216) (end 51.700005 68.004211) (width 0.25) (layer B.Cu) (net 5))
   (segment (start 52.12579 67.704212) (end 52.000004 67.704212) (width 0.25) (layer F.Cu) (net 5))
-  (segment (start 50.452001 69.252215) (end 51.700005 68.004211) (width 0.25) (layer B.Cu) (net 5))
-  (segment (start 48.095 72.54) (end 48.856999 71.778001) (width 0.25) (layer B.Cu) (net 5))
-  (segment (start 50.452001 70.521761) (end 50.452001 69.252215) (width 0.25) (layer B.Cu) (net 5))
   (segment (start 55.1 64.730002) (end 52.12579 67.704212) (width 0.25) (layer F.Cu) (net 5))
   (via (at 52.000004 67.704212) (size 0.6) (drill 0.4) (layers F.Cu B.Cu) (net 5))
-  (segment (start 51.700005 68.004211) (end 52.000004 67.704212) (width 0.25) (layer B.Cu) (net 5))
-  (segment (start 48.856999 71.778001) (end 49.195761 71.778001) (width 0.25) (layer B.Cu) (net 5))
-  (segment (start 49.195761 71.778001) (end 50.452001 70.521761) (width 0.25) (layer B.Cu) (net 5))
   (segment (start 55.700001 54.049999) (end 56 53.75) (width 0.25) (layer F.Cu) (net 5))
   (segment (start 50 62.202) (end 51.298 62.202) (width 0.25) (layer F.Cu) (net 5))
@@
   (segment (start 46.124999 55.323001) (end 46.448 55) (width 0.25) (layer F.Cu) (net 7))
   (segment (start 46.448 55) (end 47.46 55) (width 0.25) (layer F.Cu) (net 7))
+  (segment (start 53.125 57.58) (end 53.125 57.375) (width 0.6) (layer B.Cu) (net 8))
+  (segment (start 53.125 57.375) (end 49.705 53.955) (width 0.6) (layer B.Cu) (net 8))
+  (segment (start 49.705 53.955) (end 49.5 53.955) (width 0.6) (layer B.Cu) (net 8))
   (segment (start 55.715 69.015) (end 51.8 65.1) (width 0.6) (layer B.Cu) (net 8))
   (segment (start 55.715 72.54) (end 55.715 69.015) (width 0.6) (layer B.Cu) (net 8))
@@
   (segment (start 49.5 55.728613) (end 49.5 53.955) (width 0.6) (layer B.Cu) (net 8))
   (segment (start 46.378613 58.85) (end 49.5 55.728613) (width 0.6) (layer B.Cu) (net 8))
-  (segment (start 53.125 57.58) (end 52.78 57.58) (width 0.6) (layer B.Cu) (net 8))
   (segment (start 45.3 58.85) (end 46.378613 58.85) (width 0.6) (layer B.Cu) (net 8))
-  (segment (start 52.78 57.58) (end 49.5 54.3) (width 0.6) (layer B.Cu) (net 8))
-  (segment (start 49.5 54.3) (end 49.5 53.955) (width 0.6) (layer B.Cu) (net 8))
   (segment (start 54.7 57.58) (end 53.125 57.58) (width 0.6) (layer B.Cu) (net 8))
   (segment (start 49.5 53.955) (end 49.5 50.25) (width 0.6) (layer B.Cu) (net 8))
@@
   (segment (start 49.365 50.115) (end 49.5 50.25) (width 0.6) (layer F.Cu) (net 8))
   (via (at 49.5 50.25) (size 0.6) (drill 0.4) (layers F.Cu B.Cu) (net 8))
+  (segment (start 45.3 61.39) (end 46.86 61.39) (width 0.25) (layer B.Cu) (net 9))
+  (segment (start 46.86 61.39) (end 50.5 57.75) (width 0.25) (layer B.Cu) (net 9))
+  (segment (start 50.5 56.596218) (end 50.5 56.171954) (width 0.25) (layer B.Cu) (net 9))
+  (segment (start 50.5 57.75) (end 50.5 56.596218) (width 0.25) (layer B.Cu) (net 9))
+  (segment (start 50.761999 55.909955) (end 50.5 56.171954) (width 0.25) (layer F.Cu) (net 9))
+  (segment (start 50 55) (end 50.761999 55.761999) (width 0.25) (layer F.Cu) (net 9))
+  (segment (start 50.761999 55.761999) (end 50.761999 55.909955) (width 0.25) (layer F.Cu) (net 9))
+  (via (at 50.5 56.171954) (size 0.6) (drill 0.4) (layers F.Cu B.Cu) (net 9))
   (segment (start 50.2 64.383898) (end 50.2 61.4) (width 0.25) (layer B.Cu) (net 9))
   (segment (start 54.445 68.628898) (end 50.2 64.383898) (width 0.25) (layer B.Cu) (net 9))
   (segment (start 54.445 70) (end 54.445 68.628898) (width 0.25) (layer B.Cu) (net 9))
-  (segment (start 45.3 61.39) (end 50.21 61.39) (width 0.25) (layer B.Cu) (net 9))
-  (segment (start 50.21 61.39) (end 50.8 60.8) (width 0.25) (layer B.Cu) (net 9))
-  (segment (start 50.540614 56.471999) (end 50.240615 56.172) (width 0.25) (layer B.Cu) (net 9))
-  (segment (start 50.8 60.8) (end 50.8 56.731385) (width 0.25) (layer B.Cu) (net 9))
-  (segment (start 50.8 56.731385) (end 50.540614 56.471999) (width 0.25) (layer B.Cu) (net 9))
-  (segment (start 50 55) (end 50 56.07763) (width 0.25) (layer F.Cu) (net 9))
-  (segment (start 50 56.07763) (end 50.09437 56.172) (width 0.25) (layer F.Cu) (net 9))
-  (via (at 50.240615 56.172) (size 0.6) (drill 0.4) (layers F.Cu B.Cu) (net 9))
-  (segment (start 50.09437 56.172) (end 50.240615 56.172) (width 0.25) (layer F.Cu) (net 9))
   (segment (start 46.525 63.93) (end 45.3 63.93) (width 0.25) (layer B.Cu) (net 10))
   (segment (start 53.175 72.54) (end 53.175 67.995309) (width 0.25) (layer B.Cu) (net 10))
@@
   (segment (start 56.7 60.149986) (end 55.949988 60.899998) (width 0.25) (layer F.Cu) (net 16))
   (via (at 56.058051 63.558051) (size 0.6) (drill 0.4) (layers F.Cu B.Cu) (net 16))
+  (segment (start 50.635 72.54) (end 49.873001 71.778001) (width 0.25) (layer F.Cu) (net 17))
+  (segment (start 49.873001 71.778001) (end 49.028001 71.778001) (width 0.25) (layer F.Cu) (net 17))
+  (segment (start 48.100009 70.850009) (end 48.100009 68.700009) (width 0.25) (layer F.Cu) (net 17))
+  (segment (start 49.028001 71.778001) (end 48.100009 70.850009) (width 0.25) (layer F.Cu) (net 17))
   (segment (start 48.100009 68.700009) (end 48.099999 68.699999) (width 0.25) (layer F.Cu) (net 17))
-  (segment (start 48.100009 70.500009) (end 48.100009 68.700009) (width 0.25) (layer F.Cu) (net 17))
+  (segment (start 48.099999 68.699999) (end 47.8 68.4) (width 0.25) (layer F.Cu) (net 17))
   (via (at 47.8 68.4) (size 0.6) (drill 0.4) (layers F.Cu B.Cu) (net 17))
-  (segment (start 49.378001 71.778001) (end 48.100009 70.500009) (width 0.25) (layer F.Cu) (net 17))
   (segment (start 45 65.3) (end 47.8 68.1) (width 0.25) (layer B.Cu) (net 17))
-  (segment (start 50.635 72.54) (end 49.873001 71.778001) (width 0.25) (layer F.Cu) (net 17))
-  (segment (start 49.873001 71.778001) (end 49.378001 71.778001) (width 0.25) (layer F.Cu) (net 17))
-  (segment (start 48.099999 68.699999) (end 47.8 68.4) (width 0.25) (layer F.Cu) (net 17))
   (segment (start 47.8 68.1) (end 47.8 68.4) (width 0.25) (layer B.Cu) (net 17))
   (segment (start 45 65.3) (end 44.6 64.9) (width 0.25) (layer F.Cu) (net 17))

Commit message: switched reset pullups from 2K2 to 10K
Parts:
- R1: value 2K2 -> 10K
Changed lines of the file:
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@@
     (links 37)
     (no_connects 1)
-    (area 40.974999 38.3 72.135715 89.000001)
+    (area 41.924999 44.924999 58.075001 74.075001)
     (thickness 1.6)
     (drawings 27)
@@
       (effects (font (size 1 1) (thickness 0.15)) (justify mirror))
     )
-    (fp_text value 2K2 (at 0.004999 0.065 90) (layer B.SilkS)
+    (fp_text value 10K (at 0.004999 0.065 90) (layer B.SilkS)
       (effects (font (size 0.5 0.5) (thickness 0.125)) (justify mirror))
     )

Commit message: more fixes :-s
Routing:
- net /SCL_2: track 20.2 -> 23.6 mm
Changed lines of the file:
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@@
   (general
     (links 37)
-    (no_connects 1)
-    (area 41.924999 44.924999 58.075001 74.075001)
+    (no_connects 0)
+    (area 40.974999 38.3 72.135715 89.000001)
     (thickness 1.6)
     (drawings 27)
-    (tracks 279)
+    (tracks 281)
     (zones 0)
     (modules 8)
@@
   (segment (start 49.365 50.115) (end 49.5 50.25) (width 0.6) (layer F.Cu) (net 8))
   (via (at 49.5 50.25) (size 0.6) (drill 0.4) (layers F.Cu B.Cu) (net 8))
+  (segment (start 50.2 61.4) (end 50.19 61.39) (width 0.25) (layer B.Cu) (net 9))
+  (segment (start 50.19 61.39) (end 46.86 61.39) (width 0.25) (layer B.Cu) (net 9))
   (segment (start 45.3 61.39) (end 46.86 61.39) (width 0.25) (layer B.Cu) (net 9))
   (segment (start 46.86 61.39) (end 50.5 57.75) (width 0.25) (layer B.Cu) (net 9))
