File: i2c_main_power/i2c_main_power.kicad_pcb (KiCad board)
At the start: 2 copper layers, 16 x 28 mm, 16 parts, among them U1 P82B715, U2 AP2553W6

Commit message: more fixes :-s
Routing:
- net /I2C_bridge/SCL_inside: track 10.7 -> 15.4 mm
Changed lines of the file:
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@@
   (general
     (links 34)
-    (no_connects 1)
+    (no_connects 0)
     (area 33.819048 38.3 69.35 89.000001)
     (thickness 1.6)
     (drawings 40)
-    (tracks 130)
+    (tracks 134)
     (zones 0)
     (modules 16)
@@
   (segment (start 46.2 50.45) (end 46.2 48.4) (width 0.6) (layer F.Cu) (net 4))
   (segment (start 45.4 50.5) (end 46.25 50.5) (width 0.6) (layer F.Cu) (net 4))
+  (segment (start 54.55 61.5) (end 53.95 61.5) (width 0.25) (layer F.Cu) (net 5))
+  (segment (start 53.95 61.5) (end 52.85 62.6) (width 0.25) (layer F.Cu) (net 5))
+  (segment (start 52.85 62.6) (end 51.5175 62.6) (width 0.25) (layer F.Cu) (net 5))
+  (segment (start 51.5175 62.6) (end 50.635 61.7175) (width 0.25) (layer F.Cu) (net 5))
+  (segment (start 50.635 61.7175) (end 50.635 61.4) (width 0.25) (layer F.Cu) (net 5))
   (segment (start 48.095 71) (end 48.095 69.155) (width 0.25) (layer F.Cu) (net 5))
   (segment (start 48.095 69.155) (end 48.785999 68.464001) (width 0.25) (layer F.Cu) (net 5))
   (segment (start 48.785999 68.464001) (end 48.785999 63.566501) (width 0.25) (layer F.Cu) (net 5))
   (segment (start 48.785999 63.566501) (end 50.635 61.7175) (width 0.25) (layer F.Cu) (net 5))
-  (segment (start 50.635 61.7175) (end 50.635 61.4) (width 0.25) (layer F.Cu) (net 5))
   (segment (start 50.635 67.75) (end 50.635 67.4325) (width 0.25) (layer F.Cu) (net 6))
   (segment (start 50.635 67.4325) (end 52.5675 65.5) (width 0.25) (layer F.Cu) (net 6))
