File: i2c_bridge_primary/i2c_bridge_primary.sch (KiCad schematic (older format))
At the start: 6 parts, among them U2 AP2553W6

Commit message: rename of i2c_bridge_common
Connections:
- net I2C_bridge/SCL_connector renamed i2c_bridge_common/SCL_connector
- net I2C_bridge/SCL_inside renamed i2c_bridge_common/SCL_inside
- net I2C_bridge/SDA_connector renamed i2c_bridge_common/SDA_connector
- net I2C_bridge/SDA_inside renamed i2c_bridge_common/SDA_inside
Changed lines of the file:
@@
 S 3150 1050 1800 1250
 U 58E667B4
-F0 "I2C_bridge" 60
-F1 "../I2C_bridge.sch" 60
+F0 "i2c_bridge_common" 60
+F1 "../i2c_bridge_common.sch" 60
 F2 "Gnd_inside" O R 4950 2050 60
 F3 "V_inside" O R 4950 1150 60
