File: i2c_bridge_secondary/i2c_bridge_secondary.kicad_pcb (KiCad board)
At the start: 2 copper layers, 16 x 28 mm, 13 parts, among them U1 P82B715

Commit message: rename of i2c_bridge_common
Connections:
- net /I2C_bridge/SCL_connector renamed /i2c_bridge_common/SCL_connector
- net /I2C_bridge/SCL_inside renamed /i2c_bridge_common/SCL_inside
- net /I2C_bridge/SDA_connector renamed /i2c_bridge_common/SDA_connector
- net /I2C_bridge/SDA_inside renamed /i2c_bridge_common/SDA_inside
Changed lines of the file:
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@@
   (net 1 +5V)
   (net 2 GND)
-  (net 3 /I2C_bridge/SCL_connector)
-  (net 4 /I2C_bridge/SDA_connector)
-  (net 5 /I2C_bridge/SCL_inside)
-  (net 6 /I2C_bridge/SDA_inside)
+  (net 3 /i2c_bridge_common/SCL_connector)
+  (net 4 /i2c_bridge_common/SDA_connector)
+  (net 5 /i2c_bridge_common/SCL_inside)
+  (net 6 /i2c_bridge_common/SDA_inside)
   (net 7 "Net-(D3-Pad2)")
   (net_class Default "This is the default net class."
@@
     (uvia_drill 0.1)
     (add_net +5V)
-    (add_net /I2C_bridge/SCL_connector)
-    (add_net /I2C_bridge/SCL_inside)
-    (add_net /I2C_bridge/SDA_connector)
-    (add_net /I2C_bridge/SDA_inside)
+    (add_net /i2c_bridge_common/SCL_connector)
+    (add_net /i2c_bridge_common/SCL_inside)
+    (add_net /i2c_bridge_common/SDA_connector)
+    (add_net /i2c_bridge_common/SDA_inside)
     (add_net GND)
     (add_net "Net-(D3-Pad2)")
@@
     )
     (pad 1 smd rect (at -1.905 0) (size 0.9 3) (layers F.Cu F.Paste F.Mask)
-      (net 5 /I2C_bridge/SCL_inside))
+      (net 5 /i2c_bridge_common/SCL_inside))
     (pad 2 smd rect (at -0.635 0) (size 0.9 3) (layers F.Cu F.Paste F.Mask)
-      (net 6 /I2C_bridge/SDA_inside))
+      (net 6 /i2c_bridge_common/SDA_inside))
     (pad 3 smd rect (at 0.635 0) (size 0.9 3) (layers F.Cu F.Paste F.Mask)
       (net 1 +5V))
@@
       (net 2 GND))
     (pad 1 smd rect (at -0.7 0 270) (size 0.6 0.7) (layers F.Cu F.Paste F.Mask)
-      (net 3 /I2C_bridge/SCL_connector))
+      (net 3 /i2c_bridge_common/SCL_connector))
   )
   (module Diodes_SMD:SOD-523 (layer F.Cu)
@@
       (net 2 GND))
     (pad 1 smd rect (at -0.7 0) (size 0.6 0.7) (layers F.Cu F.Paste F.Mask)
-      (net 4 /I2C_bridge/SDA_connector))
+      (net 4 /i2c_bridge_common/SDA_connector))
   )
   (module SMD_Packages:SOIC-8-N (layer F.Cu)
@@
       (net 1 +5V))
     (pad 7 smd rect (at -0.635 -3.175) (size 0.508 1.143) (layers F.Cu F.Paste F.Mask)
-      (net 3 /I2C_bridge/SCL_connector))
+      (net 3 /i2c_bridge_common/SCL_connector))
     (pad 6 smd rect (at 0.635 -3.175) (size 0.508 1.143) (layers F.Cu F.Paste F.Mask)
-      (net 5 /I2C_bridge/SCL_inside))
+      (net 5 /i2c_bridge_common/SCL_inside))
     (pad 5 smd rect (at 1.905 -3.175) (size 0.508 1.143) (layers F.Cu F.Paste F.Mask))
     (pad 4 smd rect (at 1.905 3.175) (size 0.508 1.143) (layers F.Cu F.Paste F.Mask)
       (net 2 GND))
     (pad 3 smd rect (at 0.635 3.175) (size 0.508 1.143) (layers F.Cu F.Paste F.Mask)
-      (net 6 /I2C_bridge/SDA_inside))
+      (net 6 /i2c_bridge_common/SDA_inside))
     (pad 2 smd rect (at -0.635 3.175) (size 0.508 1.143) (layers F.Cu F.Paste F.Mask)
-      (net 4 /I2C_bridge/SDA_connector))
+      (net 4 /i2c_bridge_common/SDA_connector))
     (pad 1 smd rect (at -1.905 3.175) (size 0.508 1.143) (layers F.Cu F.Paste F.Mask))
     (model SMD_Packages.3dshapes/SOIC-8-N.wrl
@@
     (fp_line (start -0.6 -0.875) (end 0.6 -0.875) (layer F.SilkS) (width 0.15))
     (pad 1 smd rect (at -0.95 0) (size 0.7 1.3) (layers F.Cu F.Paste F.Mask)
-      (net 3 /I2C_bridge/SCL_connector))
+      (net 3 /i2c_bridge_common/SCL_connector))
     (pad 2 smd rect (at 0.95 0) (size 0.7 1.3) (layers F.Cu F.Paste F.Mask)
       (net 1 +5V))
@@
     (fp_line (start -0.6 -0.875) (end 0.6 -0.875) (layer F.SilkS) (width 0.15))
     (pad 1 smd rect (at -0.95 0) (size 0.7 1.3) (layers F.Cu F.Paste F.Mask)
-      (net 4 /I2C_bridge/SDA_connector))
+      (net 4 /i2c_bridge_common/SDA_connector))
     (pad 2 smd rect (at 0.95 0) (size 0.7 1.3) (layers F.Cu F.Paste F.Mask)
       (net 1 +5V))
@@
     (fp_line (start -0.6 -0.875) (end 0.6 -0.875) (layer F.SilkS) (width 0.15))
     (pad 1 smd rect (at -0.95 0) (size 0.7 1.3) (layers F.Cu F.Paste F.Mask)
-      (net 5 /I2C_bridge/SCL_inside))
+      (net 5 /i2c_bridge_common/SCL_inside))
     (pad 2 smd rect (at 0.95 0) (size 0.7 1.3) (layers F.Cu F.Paste F.Mask)
       (net 1 +5V))
@@
     (fp_line (start -0.6 -0.875) (end 0.6 -0.875) (layer F.SilkS) (width 0.15))
     (pad 1 smd rect (at -0.95 0) (size 0.7 1.3) (layers F.Cu F.Paste F.Mask)
-      (net 6 /I2C_bridge/SDA_inside))
+      (net 6 /i2c_bridge_common/SDA_inside))
     (pad 2 smd rect (at 0.95 0) (size 0.7 1.3) (layers F.Cu F.Paste F.Mask)
       (net 1 +5V))
@@
     (pad "" thru_hole circle (at 11.5 0 270) (size 2 2) (drill 1.6) (layers *.Cu *.Mask F.SilkS))
     (pad 4 smd rect (at 3.4 3.8 270) (size 2.2 2.8) (layers F.Cu F.Paste F.Mask)
-      (net 4 /I2C_bridge/SDA_connector))
+      (net 4 /i2c_bridge_common/SDA_connector))
     (pad 2 smd rect (at 12.8 3.8 270) (size 2.8 2.8) (layers F.Cu F.Paste F.Mask)
       (net 7 "Net-(D3-Pad2)"))
     (pad 3 smd rect (at 5.3 -3.8 270) (size 2.2 2.8) (layers F.Cu F.Paste F.Mask)
-      (net 3 /I2C_bridge/SCL_connector))
+      (net 3 /i2c_bridge_common/SCL_connector))
     (pad 1 smd rect (at 0.6 3.8 270) (size 2 2.8) (layers F.Cu F.Paste F.Mask)
       (net 2 GND))

Commit message: added YamseK logo :-)
Parts:
- added svg2mod: G***, myComponents:logo, B.Cu at (50.0, 64.2)
Other:
- board text added: "i2c_bridge_secondary 2017-04-09"

Commit message: tweaks to the logo
Parts:
- moved svg2mod 6.60 mm to (50.0, 70.8)
