File: matrix_attiny861a/matrix_attiny861a.sch (KiCad schematic (older format))
At the start: 8 parts, among them IC1 ATTINY861A-S

Commit message: bugfixes preparing first order to oshpark
Parts:
- added C2: 0.1µF, Capacitors_SMD:C_0805, symbol C
Connections:
- net +5V: now also C2.1
- net GND: now also C2.2
