File: matrix_mcp23017/matrix_mcp23017.kicad_pcb (KiCad board)
At the start: 2 copper layers, 16 x 29 mm, 10 parts, among them U4 MCP23017

Commit message: added YamseK logo :-)
Parts:
- added svg2mod: G***, myComponents:logo, F.Cu at (44.0, 57.0)
Other:
- board text added: "matrix mcp23017 2017-04-09"

Commit message: tweaks to the logo
Parts:
- moved svg2mod 2.00 mm to (44.0, 55.0)
Routing:
- net GND: track 43.5 -> 52.0 mm
