File: matrix_mcp23017/matrix_mcp23017.sch (KiCad schematic (older format))
At the start: 10 parts, among them U4 MCP23017

Commit message: bugfixes preparing first order to oshpark
Connections:
- no-connect marks 2 -> 5
Changed lines of the file:
@@
 EESchema Schematic File Version 2
-LIBS:mcp23017_breakout-rescue
 LIBS:power
 LIBS:device
@@
 LIBS:valves
 LIBS:myComponents
-LIBS:mcp23017_breakout-cache
+LIBS:matrix_mcp23017-cache
 EELAYER 25 0
 EELAYER END
@@
 Connection ~ 3000 4100
 Connection ~ 3000 4500
+NoConn ~ 5000 3650
+NoConn ~ 5000 4450
+NoConn ~ 5000 4550
 $EndSCHEMATC
